Commit message: stable version

File: urdf/soft_digit_description.urdf (robot description, URDF)
Before this commit: robot digit_sensor, 4 links, 3 joints
Joints:
- joint attach: limit effort=1 velocity=20 -> (none); origin xyz=5.2041704279304212832e-18 -0.011792651350691449319 -0.0283500000000000002 rpy=0 -0 0 -> xyz=5.2041704279304212832e-18 -0.011792651350691449319 -0.0283500000000000002 rpy=0 0 0
