Commit message: add indenter controllers

File: urdf/indenters/ball_indenter.urdf (robot description, URDF)
Before this commit: robot digit, 2 links, 1 joints
Joints:
- joint rail: axis 0 0 1 -> 0 1 0; limit lower=0.15 upper=0.161 -> lower=0.0 upper=0.2

File: urdf/sensor/digit_sensor.urdf (robot description, URDF)
Before this commit: robot digit, 2 links, 1 joints
Links:
- added link world
Joints:
- added joint world_digit: type fixed, parent world, child digit_base, origin xyz=0 0 0 rpy=1.57079632 0 0, axis 0 0 0
